Commit message: implemented force controlled unscrewing

File: emo_demonstration/urdf/screw_driver_addon.urdf (robot description, URDF)
Before this commit: robot endeffector, 3 links, 2 joints
Links:
- link screw_tip: geometry visual sphere radius=0.0005
- link screwdriver: geometry collision mesh filename=endeffector_mesh/Schrauber.stl scale=0.001 0.001 0.001; visual mesh filename=endeffector_mesh/Schrauber.stl scale=0.001 0.001 0.001
