Commit message: deleted screw from endeffector to prevent duplicate mehes

File: emo_demonstration/urdf/endeffector.urdf (robot description, URDF)
Before this commit: robot endeffector, 6 links, 5 joints
Links:
- link screwdriver: geometry 

Commit message: d_emo_nstration V0.9 complet
full disassembly sequence implemented

File: emo_demonstration/urdf/endeffector.urdf (robot description, URDF)
Before this commit: robot endeffector, 6 links, 5 joints
Links:
- link gripper_center_link: geometry visual sphere radius=0.005
- link screw_tip: geometry 
Joints:
- joint left_jaw: limit lower=0 upper=0.01 effort=1000 velocity=0.01 -> lower=0 upper=0.01 effort=1 velocity=0.01
- joint right_jaw: limit lower=0 upper=0.01 effort=1000 velocity=0.01 -> lower=0 upper=0.01 effort=1 velocity=0.01
- joint screwdriver_joint: origin xyz=0.089 -0.104 0.032 rpy=0 0 0 -> xyz=0.083 -0.104 0.026 rpy=0 0 0

File: emo_demonstration/urdf/screw_driver_addon.urdf (robot description, URDF)
Before this commit: robot endeffector, 3 links, 2 joints
Links:
- link screw_tip: geometry collision sphere radius=0.002; visual sphere radius=0.002
- link screwdriver: geometry visual mesh filename=endeffector_mesh/Schrauber.stl scale=0.001 0.001 0.001
Joints:
- joint base_joint: origin xyz=0 0 0 rpy=0 0 0 -> xyz=-0.006 0.0 -0.006 rpy=0 0 0
- joint screwdriver_joint: origin xyz=0.089 -0.104 0.032 rpy=0 0 0 -> xyz=0.083 -0.10 0.026 rpy=0 0 0
