Commit message: milling complete

File: emo_demonstration/urdf/milling_addon.urdf (robot description, URDF)
Before this commit: robot endeffector, 4 links, 3 joints
Joints:
- joint mill_joint: origin xyz=-0.106 0.125 0.028 rpy=0 0 0 -> xyz=-0.1055 0.12 0.0265 rpy=0 0 0
- joint mill_joint2: origin xyz=-0.106 0.125 0.028 rpy=0 0 0 -> xyz=-0.1055 0.12 0.027 rpy=0 0 0
